Commit message: integrated the imu

File: jidenna_description/urdf/jidenna_ros2_control.urdf.xacro (robot description, xacro)
@@ -18,4 +18,5 @@
             </hardware>
         </xacro:unless>
+        <!-- ===================== Wheel joints ===================== -->
         <joint name="left_wheel_joint">
             <command_interface name="velocity">
@@ -34,4 +35,20 @@
             <state_interface name="position"/>
         </joint>
+        <!-- ===================== IMU sensor ======================= -->
+        <!--
+          Note: <sensor> is a sibling of <joint>, not a child of <hardware>.
+          Only export it for real hardware (the sim's IMU comes from Gazebo).
+        -->
+        <xacro:unless value="$(arg is_sim)">
+            <sensor name="imu_sensor">
+                <state_interface name="orientation.x"/>
+                <state_interface name="orientation.y"/>
+                <state_interface name="orientation.z"/>
+                <state_interface name="orientation.w"/>
+                <state_interface name="angular_velocity.x"/>
+                <state_interface name="angular_velocity.y"/>
+                <state_interface name="angular_velocity.z"/>
+            </sensor>
+        </xacro:unless>
     </ros2_control>
 </robot>
